Commit message: Fixed laser 3d model

File: etfsa_atv_description/urdf/accessories/sick_lms1xx_mount.urdf.xacro (robot description, xacro)
@@ -19,5 +19,5 @@
     </link>
     <joint name="${prefix}_laser_joint" type="fixed">
-      <origin xyz="0.0352 0 0.0566" rpy="${M_PI} 0 0" />
+      <origin xyz="0.0352 0 0.1566" rpy="0 0 0" />
       <parent link="${prefix}_laser_mount" />
       <child link="${prefix}_laser" />
